Commit message: Bullet migration: checkpoint

File: pioneer/robot/assets/pioneer.urdf (robot description, URDF)
Before this commit: robot pioneer, 5 links, 4 joints
Links:
- added link robot:arm2, mass 1.0; visual box size=10 1 2
- added link robot:hinge2, mass 1.0; visual box size=2 0.5 1
- added link robot:rotator2, mass 1.0; visual cylinder length=0.4 radius=1
Joints:
- added joint robot:arm1_to_arm2: type revolute, parent robot:arm1, child robot:arm2, origin xyz=0 0 11, axis 0 1 0, limit lower=-1.309 upper=1.309 effort=1.0
- added joint robot:arm2_to_rotator2: type revolute, parent robot:arm2, child robot:rotator2, origin xyz=0 1 0, axis 1 0 0, limit lower=-3.1416 upper=3.1416 effort=1.0
- added joint robot:rotator2_to_hinge2: type fixed, parent robot:rotator2, child robot:hinge2
- joint robot:base_to_rotator1: limit lower=-1.309 upper=1.309 effort=1.0 -> lower=-3.1416 upper=3.1416 effort=1.0

Commit message: Bullet migration: updated pioneer URDF model

File: pioneer/robot/assets/pioneer.urdf (robot description, URDF)
Before this commit: robot pioneer, 8 links, 7 joints
Links:
- added link robot:arm3, mass 1.0; visual box size=3 0.5 1; visual box size=3 0.5 1
- added link robot:effector, mass 1.0; visual box size=0.2 0.2 2.5; visual box size=1.0 0.2 0.2
- added link robot:pointer, mass 1.0; visual sphere radius=0.2
- added link robot:rotator3, mass 1.0; visual cylinder length=0.4 radius=1
Joints:
- added joint robot:arm3_to_rotator3: type revolute, parent robot:arm3, child robot:rotator3, origin xyz=0 0 0, axis 1 0 0, limit lower=-3.1416 upper=3.1416 effort=1.0
- added joint robot:effector_to_pointer: type fixed, parent robot:effector, child robot:pointer
- added joint robot:hinge2_to_arm3: type revolute, parent robot:hinge2, child robot:arm3, origin xyz=11 0 0, axis 0 1 0, limit lower=-1.5708 upper=1.5708 effort=1.0
- added joint robot:rotator3_to_effector: type fixed, parent robot:rotator3, child robot:effector
