Commit message: Bullet migration: pioneer action and observation

File: pioneer/envs/pioneer/assets/pioneer_6dof.urdf (robot description, URDF)
Before this commit: robot pioneer, 12 links, 11 joints
Links:
- added link target, mass 1.0; visual sphere radius=0.2
Joints:
- added joint world_to_target: type fixed, parent world, child target

Commit message: Fixed some URDFs...

File: pioneer/envs/pioneer/assets/pioneer_6dof.urdf (robot description, URDF)
Before this commit: robot pioneer, 13 links, 12 joints
Joints:
- joint robot:effector_to_pointer: origin (none) -> xyz=3.6 0 1.9
- joint world_to_target: origin (none) -> xyz=20 -5 4

Commit message: Added some collision modelling

File: pioneer/envs/pioneer/assets/pioneer_6dof.urdf (robot description, URDF)
Before this commit: robot pioneer, 12 links, 11 joints
Links:
- link robot:arm1: geometry collision box size=12 1 2; visual box size=12 1 2
- link robot:arm2: geometry collision box size=10 1 2; visual box size=10 1 2
- link robot:arm3: geometry collision box size=3 0.5 1; collision box size=3 0.5 1
- link robot:effector: geometry collision box size=0.2 0.2 2.5; collision box size=1.0 0.2 0.2
- link robot:hinge1: geometry collision box size=2 1 2; collision box size=2 1 2
- link robot:hinge2: geometry collision box size=2 0.5 1; visual box size=2 0.5 1
- link robot:pointer: geometry collision sphere radius=0.2; visual sphere radius=0.2
- link robot:rotator1: geometry collision cylinder length=1 radius=4; visual cylinder length=1 radius=4
- link robot:rotator2: geometry collision cylinder length=0.4 radius=1; visual cylinder length=0.4 radius=1
- link robot:rotator3: geometry collision cylinder length=0.4 radius=1; visual cylinder length=0.4 radius=1

Commit message: Added randomized obstacle generation

File: pioneer/envs/pioneer/assets/pioneer_6dof.urdf (robot description, URDF)
Before this commit: robot pioneer, 12 links, 11 joints
Links:
- added link ground, mass 10.0; collision box size=200 200 1; visual box size=200 200 1
Joints:
- added joint world_to_ground: type fixed, parent world, child ground

Commit message: Reduced ground size

File: pioneer/envs/pioneer/assets/pioneer_6dof.urdf (robot description, URDF)
Before this commit: robot pioneer, 13 links, 12 joints
Links:
- link ground: geometry collision box size=60 60 0.2; visual box size=60 60 0.2

Commit message: Scaled the model down 10x, added light source for rendering

File: pioneer/envs/pioneer/assets/pioneer_6dof.urdf (robot description, URDF)
Before this commit: robot pioneer, 13 links, 12 joints
Links:
- link ground: geometry collision box size=6 6 0.2; visual box size=6 6 0.2
- link robot:arm1: geometry collision box size=1.2 0.1 0.2; visual box size=1.2 0.1 0.2
- link robot:arm2: geometry collision box size=1 0.1 0.2; visual box size=1 0.1 0.2
- link robot:arm3: geometry collision box size=0.3 0.05 0.1; collision box size=0.3 0.05 0.1
- link robot:effector: geometry collision box size=0.02 0.02 0.25; collision box size=0.1 0.02 0.02
- link robot:hinge1: geometry collision box size=0.2 0.1 0.2; collision box size=0.2 0.1 0.2
- link robot:hinge2: geometry collision box size=0.2 0.05 0.1; visual box size=0.2 0.05 0.1
- link robot:pointer: geometry collision sphere radius=0.02; visual sphere radius=0.02
- link robot:rotator1: geometry collision cylinder length=0.1 radius=0.4; visual cylinder length=0.1 radius=0.4
- link robot:rotator2: geometry collision cylinder length=0.04 radius=0.1; visual cylinder length=0.04 radius=0.1
- link robot:rotator3: geometry collision cylinder length=0.04 radius=0.1; visual cylinder length=0.04 radius=0.1
Joints:
- joint robot:arm1_to_arm2: origin xyz=0 0 11 -> xyz=0 0 1.1
- joint robot:arm2_to_rotator2: origin xyz=0 1 0 -> xyz=0 0.1 0
- joint robot:effector_to_pointer: origin xyz=3.6 0 1.9 -> xyz=0.36 0 0.19
- joint robot:hinge1_to_arm1: origin xyz=0 0 3 -> xyz=0 0 0.3
- joint robot:hinge2_to_arm3: origin xyz=11 0 0 -> xyz=1.1 0 0
